File: Cessna172NavCom/Cessna 172 nav and com radio.kicad_pcb (KiCad board)
At the start: 2 copper layers, 330.2 x 76.2 mm, 46 parts, among them J1 Conn_02x12_Odd_Even, SW1 COMM toggle, SW1 COMM transfer switch, SW2 NAV toggle, SW2 NAV transfer switch, SW3 Tuning encoder, SW4 Tuning encoder, SW5 Test switch, SW6 Ident switch, U1 MAX7219 COM standby, U2 MAX7219 COM standby, U3 MAX7219 COM standby, U4 MAX7219 COM standby

Commit message: Traces for one LCD bank complete
Parts:
- removed the SW1 at (58.1, 84.9)
- removed the SW1 at (127.0, 55.9)
- removed the SW2 at (67.8, 84.9)
- removed the SW2 at (275.6, 55.9)
- added C1: 10uF, Capacitor_THT:CP_Radial_D5.0mm_P2.00mm, F.Cu at (215.5, 199.2)
- added C10: 0.1uf, Capacitor_SMD:C_0805_2012Metric_Pad1.15x1.40mm_HandSolder, F.Cu at (226.9, 212.9)
- added C11: 0.1uf, Capacitor_SMD:C_0805_2012Metric_Pad1.15x1.40mm_HandSolder, F.Cu at (231.7, 209.9)
- added C2: 0.1uF, Capacitor_SMD:C_0805_2012Metric_Pad1.15x1.40mm_HandSolder, B.Cu at (109.0, 69.1)
- added C3: 0.1uF, Capacitor_SMD:C_0805_2012Metric_Pad1.15x1.40mm_HandSolder, B.Cu at (143.8, 113.0)
- added C4: 0.1uF, Capacitor_SMD:C_0805_2012Metric_Pad1.15x1.40mm_HandSolder, B.Cu at (210.3, 71.9)
- added C5: 0.1uF, Capacitor_SMD:C_0805_2012Metric_Pad1.15x1.40mm_HandSolder, B.Cu at (213.1, 110.4)
- added D1: LED, LED_SMD:LED_0805_2012Metric_Pad1.15x1.40mm_HandSolder, F.Cu at (222.2, 197.5)
- added R1: 220, Resistor_SMD:R_0805_2012Metric_Pad1.15x1.40mm_HandSolder, F.Cu at (222.2, 200.5)
- added R13: 220, Resistor_SMD:R_0805_2012Metric_Pad1.15x1.40mm_HandSolder, F.Cu at (226.9, 197.4)
- added R14: 10k, Resistor_SMD:R_0805_2012Metric_Pad1.15x1.40mm_HandSolder, F.Cu at (222.2, 212.9)
- added R15: 10k, Resistor_SMD:R_0805_2012Metric_Pad1.15x1.40mm_HandSolder, F.Cu at (226.9, 209.9)
- added R16: 10k, Resistor_SMD:R_0805_2012Metric_Pad1.15x1.40mm_HandSolder, F.Cu at (222.2, 209.9)
- added R17: 10k, Resistor_SMD:R_0805_2012Metric_Pad1.15x1.40mm_HandSolder, F.Cu at (222.2, 215.8)
- added SW1: COMM toggle, Cessna 172 nav and com radio:B3W-9000-xxx, F.Cu at (244.9, 178.2)
- added SW2: NAV toggle, Cessna 172 nav and com radio:B3W-9000-xxx, F.Cu at (231.0, 190.0)
- added SW7: Tuning encoder, Cessna 172 nav and com radio:EN11-HSM1BF20, F.Cu at (213.0, 218.7)
- J1, RV1: moved to F.Cu
- LED1, LED11, LED16, LED6: value MobiFlight digit 5 -> MobiFlight digit 4
- LED10, LED15, LED20, LED5: value Mobiflight digit 0 -> Mobiflight digit 8
- LED12, LED17, LED2, LED7: value MobiFlight digit 4 -> MobiFlight digit 5
- LED13, LED18, LED3, LED8: value MobiFlight digit 2 -> MobiFlight digit 6
- LED14, LED19, LED4, LED9: value MobiFlight digit 1 -> MobiFlight digit 7
- moved SW4 201.0 mm to (149.1, 155.9)
- moved RV1 173.6 mm to (215.1, 180.8)
- moved LED20 164.0 mm to (175.3, 113.2)
- moved LED17 140.5 mm to (213.4, 113.2)
- moved J1 136.6 mm to (208.3, 174.5), turned to 0 degrees
- moved U4 129.0 mm to (200.7, 113.2)
- moved LED19 129.0 mm to (188.0, 113.2)
- moved SW3 107.5 mm to (109.4, 155.9)
- moved LED16 106.9 mm to (226.1, 113.2)
- moved LED18 106.9 mm to (200.7, 113.2)
- moved SW5 102.3 mm to (219.1, 190.0)
- moved SW6 98.3 mm to (233.0, 178.2)
- moved LED5 87.6 mm to (160.0, 70.6)
- moved LED9 81.9 mm to (109.2, 113.2)
- moved R8 80.1 mm to (118.6, 153.1), turned to 0 degrees
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Connections:
- J1 pad 19: COMM_VOL_SW -> IDENT_SW
- J1 pad 21: IDENT_SW -> IDENT_LED
- J1 pad 23: IDENT_LED -> Net-(J1-Pad23)
- LED1 pad 3: Net-(LED1-Pad3) -> /5 digit LCD display/DIG_4
- LED1 pad 8: /5 digit LCD display/DIG_4 -> Net-(LED1-Pad8)
- LED10 pad 3: Net-(LED10-Pad3) -> /sheet5F611637/DIG_0
- LED10 pad 8: /sheet5F611637/DIG_0 -> Net-(LED10-Pad8)
- LED11 pad 3: Net-(LED11-Pad3) -> /sheet5F613960/DIG_4
- LED11 pad 8: /sheet5F613960/DIG_4 -> Net-(LED11-Pad8)
- LED12 pad 3: Net-(LED12-Pad3) -> /sheet5F613960/DIG_3
- LED12 pad 8: /sheet5F613960/DIG_3 -> Net-(LED12-Pad8)
- LED13 pad 3: Net-(LED13-Pad3) -> /sheet5F613960/DIG_2
- LED13 pad 8: /sheet5F613960/DIG_2 -> Net-(LED13-Pad8)
- LED14 pad 3: Net-(LED14-Pad3) -> /sheet5F613960/DIG_1
- LED14 pad 8: /sheet5F613960/DIG_1 -> Net-(LED14-Pad8)
- LED15 pad 3: Net-(LED15-Pad3) -> /sheet5F613960/DIG_0
- LED15 pad 8: /sheet5F613960/DIG_0 -> Net-(LED15-Pad8)
- LED16 pad 3: Net-(LED16-Pad3) -> /sheet5F613961/DIG_4
- LED16 pad 8: /sheet5F613961/DIG_4 -> Net-(LED16-Pad8)
- LED17 pad 3: Net-(LED17-Pad3) -> /sheet5F613961/DIG_3
- LED17 pad 8: /sheet5F613961/DIG_3 -> Net-(LED17-Pad8)
- LED18 pad 3: Net-(LED18-Pad3) -> /sheet5F613961/DIG_2
- LED18 pad 8: /sheet5F613961/DIG_2 -> Net-(LED18-Pad8)
- LED19 pad 3: Net-(LED19-Pad3) -> /sheet5F613961/DIG_1
- LED19 pad 8: /sheet5F613961/DIG_1 -> Net-(LED19-Pad8)
- LED2 pad 3: Net-(LED2-Pad3) -> /5 digit LCD display/DIG_3
- LED2 pad 8: /5 digit LCD display/DIG_3 -> Net-(LED2-Pad8)
- LED20 pad 3: Net-(LED20-Pad3) -> /sheet5F613961/DIG_0
- LED20 pad 8: /sheet5F613961/DIG_0 -> Net-(LED20-Pad8)
- LED3 pad 3: Net-(LED3-Pad3) -> /5 digit LCD display/DIG_2
- LED3 pad 8: /5 digit LCD display/DIG_2 -> Net-(LED3-Pad8)
- LED4 pad 3: Net-(LED4-Pad3) -> /5 digit LCD display/DIG_1
- LED4 pad 8: /5 digit LCD display/DIG_1 -> Net-(LED4-Pad8)
- LED5 pad 3: Net-(LED5-Pad3) -> /5 digit LCD display/DIG_0
- LED5 pad 8: /5 digit LCD display/DIG_0 -> Net-(LED5-Pad8)
- LED6 pad 3: Net-(LED6-Pad3) -> /sheet5F611637/DIG_4
- LED6 pad 8: /sheet5F611637/DIG_4 -> Net-(LED6-Pad8)
- LED7 pad 3: Net-(LED7-Pad3) -> /sheet5F611637/DIG_3
- LED7 pad 8: /sheet5F611637/DIG_3 -> Net-(LED7-Pad8)
- LED8 pad 3: Net-(LED8-Pad3) -> /sheet5F611637/DIG_2
- LED8 pad 8: /sheet5F611637/DIG_2 -> Net-(LED8-Pad8)
- LED9 pad 3: Net-(LED9-Pad3) -> /sheet5F611637/DIG_1
- LED9 pad 8: /sheet5F611637/DIG_1 -> Net-(LED9-Pad8)
Routing:
- net /5 digit LCD display/SEG_D: track 0.00 -> 115.0 mm, vias 0 -> 5
- net /5 digit LCD display/SEG_E: track 0.00 -> 105.8 mm, vias 0 -> 5
- net /5 digit LCD display/SEG_DP: track 0.00 -> 105.0 mm, vias 0 -> 1
- net /5 digit LCD display/SEG_C: track 0.00 -> 95.8 mm, vias 0 -> 6
- net /5 digit LCD display/SEG_F: track 0.00 -> 81.2 mm, vias 0 -> 5
- net /5 digit LCD display/SEG_G: track 0.00 -> 79.9 mm, vias 0 -> 4
- net /5 digit LCD display/SEG_A: track 0.00 -> 72.4 mm, vias 0 -> 4
- net /5 digit LCD display/SEG_B: track 0.00 -> 68.7 mm
- net /5 digit LCD display/DIG_0: track 0.00 -> 44.1 mm
- net /5 digit LCD display/DIG_1: track 0.00 -> 38.1 mm
- net /5 digit LCD display/DIG_2: track 0.00 -> 21.3 mm, vias 0 -> 1
- net +5V: track 0.00 -> 12.3 mm, vias 0 -> 1
- net LOAD: track 0.00 -> 12.2 mm
- net /5 digit LCD display/DIG_4: track 0.00 -> 12.1 mm, vias 0 -> 1
- net CLK: track 0.00 -> 12.0 mm
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Other:
- board outline removed

Commit message: First full layout attempt, new 3D models
Parts:
- removed R13: 220, Resistor_SMD:R_0805_2012Metric_Pad1.15x1.40mm_HandSolder
- removed SW5: Test switch, Cessna 172 nav and com radio:B3W-9000-xxx
- added D2: LED, LED_SMD:LED_0805_2012Metric_Pad1.15x1.40mm_HandSolder, B.Cu at (41.7, 64.4)
- added J2: Conn_01x05, Connector_PinHeader_2.54mm:PinHeader_1x05_P2.54mm_Vertical, B.Cu at (188.7, 59.4)
- added J3: Barrel_Jack_MountingPin, Cessna 172 nav and com radio:BarrelJack_Horizontal, B.Cu at (35.2, 57.7)
- added R2: 220k, Resistor_SMD:R_0805_2012Metric_Pad1.15x1.40mm_HandSolder, F.Cu at (82.6, 73.6)
- added R3: 220k, Resistor_SMD:R_0805_2012Metric_Pad1.15x1.40mm_HandSolder, B.Cu at (44.1, 64.5)
- C1, J1, RV1: moved to B.Cu
- D1: footprint LED_SMD:LED_0805_2012Metric_Pad1.15x1.40mm_HandSolder -> LED_THT:LED_D5.0mm
- R1: value 220 -> 220k; moved to B.Cu
- moved C1 222.2 mm to (44.1, 57.7)
- moved C10 221.5 mm to (54.7, 73.6), turned to 90 degrees
- moved R14 220.6 mm to (51.1, 73.6), turned to 90 degrees
- moved SW7 218.1 mm to (60.8, 62.6)
- moved C11 214.1 mm to (66.6, 73.6), turned to 270 degrees
- moved R17 213.3 mm to (63.2, 73.6), turned to 270 degrees
- moved R16 213.2 mm to (58.2, 73.6), turned to 90 degrees
- moved R15 207.8 mm to (70.2, 73.6), turned to 270 degrees
- moved SW1 193.0 mm to (93.7, 58.2)
- moved D1 191.2 mm to (82.6, 66.9), turned to 270 degrees
- moved SW4 166.5 mm to (287.0, 62.5)
- moved R10 158.0 mm to (296.6, 73.6), turned to 270 degrees
- moved C9 156.5 mm to (293.2, 73.6), turned to 270 degrees
- moved J1 153.3 mm to (110.0, 56.8), turned to 270 degrees
- moved R12 150.4 mm to (289.5, 73.6), turned to 270 degrees
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Connections:
- net Net-(C11-Pad1) renamed /sheet5F5E0D6C/B
- net Net-(C7-Pad1) renamed /Tuning rotary encoder and switch/B
- net Net-(C9-Pad1) renamed /sheet5F5DD32A/B
- C10 pad 2: Net-(C10-Pad2) -> /sheet5F5E0D6C/A
- C6 pad 2: Net-(C6-Pad2) -> /Tuning rotary encoder and switch/A
- C8 pad 2: Net-(C8-Pad2) -> /sheet5F5DD32A/A
- D1 pad 1: +5V -> GND
- D1 pad 2: +5V -> Net-(D1-Pad2)
- R11 pad 1: NAV_RIGHT -> NAV_LEFT
- R11 pad 2: Net-(C8-Pad2) -> /sheet5F5DD32A/A
- R12 pad 2: NAV_LEFT -> NAV_RIGHT
- R14 pad 1: Net-(C10-Pad2) -> +5V
- R14 pad 2: +5V -> /sheet5F5E0D6C/A
- R16 pad 1: COMM_VOL_RIGHT -> COMM_VOL_LEFT
- R16 pad 2: Net-(C10-Pad2) -> /sheet5F5E0D6C/A
- R17 pad 2: COMM_VOL_LEFT -> COMM_VOL_RIGHT
- R5 pad 1: Net-(C6-Pad2) -> +5V
- R5 pad 2: +5V -> /Tuning rotary encoder and switch/A
- R7 pad 1: COMM_RIGHT -> COMM_LEFT
- R7 pad 2: Net-(C6-Pad2) -> /Tuning rotary encoder and switch/A
- R8 pad 2: COMM_LEFT -> COMM_RIGHT
- R9 pad 1: Net-(C8-Pad2) -> +5V
- R9 pad 2: +5V -> /sheet5F5DD32A/A
- SW3 pad A: Net-(C6-Pad2) -> /Tuning rotary encoder and switch/A
- SW4 pad A: Net-(C8-Pad2) -> /sheet5F5DD32A/A
- SW7 pad A: Net-(C10-Pad2) -> /sheet5F5E0D6C/A
- U4 pad 24: /sheet5F613961/DOUT -> DOUT
Routing:
- net /sheet5F611637/SEG_D: track 0.00 -> 115.0 mm, vias 0 -> 5
- net /sheet5F613960/SEG_D: track 0.00 -> 115.0 mm, vias 0 -> 5
- net /sheet5F613961/SEG_D: track 0.00 -> 115.0 mm, vias 0 -> 5
- net /sheet5F613961/SEG_E: track 0.00 -> 105.8 mm, vias 0 -> 5
- net /sheet5F613960/SEG_E: track 0.00 -> 105.8 mm, vias 0 -> 5
- net /sheet5F611637/SEG_E: track 0.00 -> 105.8 mm, vias 0 -> 5
- net /sheet5F613961/SEG_DP: track 0.00 -> 105.0 mm, vias 0 -> 1
- net /sheet5F611637/SEG_DP: track 0.00 -> 105.0 mm, vias 0 -> 1
- net /sheet5F613960/SEG_DP: track 0.00 -> 105.0 mm, vias 0 -> 1
- net /sheet5F611637/SEG_C: track 0.00 -> 95.8 mm, vias 0 -> 6
- net /sheet5F613961/SEG_C: track 0.00 -> 95.8 mm, vias 0 -> 6
- net /sheet5F613960/SEG_C: track 0.00 -> 95.8 mm, vias 0 -> 6
- net /sheet5F611637/SEG_F: track 0.00 -> 81.2 mm, vias 0 -> 5
- net /sheet5F613961/SEG_F: track 0.00 -> 81.2 mm, vias 0 -> 5
- net /sheet5F613960/SEG_F: track 0.00 -> 81.2 mm, vias 0 -> 5
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- added copper zone on B.Cu, net GND
- added copper zone on F.Cu, net GND
Other:
- board outline added: 289 x 69 mm
- net class +5V added: clearance 0.2, trace_width 1.016, via_dia 0.8, via_drill 0.4
- net class GND added: clearance 0.2, trace_width 1.016, via_dia 0.8, via_drill 0.4
- board text added: "COMM active"
- board text added: "COMM encoder"
- board text added: "COMM standby"
- board text added: "COMM test LED"
- board text added: "COMM volume encoder"
- board text added: "NAV active"
- board text added: "NAV encoder"
- board text added: "NAV standby"

Commit message: Re-work to use 5 digit LEDs
Parts:
- removed LED1, LED11, LED16, LED6: MobiFlight digit 4, Cessna 172 nav and com radio:KYX-5101AS
- removed LED10, LED15, LED20, LED5: Mobiflight digit 8, Cessna 172 nav and com radio:KYX-5101AS
- removed LED12, LED17, LED2, LED7: MobiFlight digit 5, Cessna 172 nav and com radio:KYX-5101AS
- removed LED13, LED18, LED3, LED8: MobiFlight digit 6, Cessna 172 nav and com radio:KYX-5101AS
- removed LED14, LED19, LED4, LED9: MobiFlight digit 7, Cessna 172 nav and com radio:KYX-5101AS
- removed R17: 10k, Resistor_SMD:R_0805_2012Metric_Pad1.15x1.40mm_HandSolder
- removed SW7: Tuning encoder, Cessna 172 nav and com radio:EN11-HSM1BF20
- added D3: LED, LED_THT:LED_D5.0mm, F.Cu at (59.3, 69.6)
- added R13: 10k, Resistor_SMD:R_0805_2012Metric_Pad1.15x1.40mm_HandSolder, F.Cu at (108.8, 66.0)
- added R4: 220k, Resistor_SMD:R_0805_2012Metric_Pad1.15x1.40mm_HandSolder, B.Cu at (119.4, 68.8)
- added SW5: Tuning encoder, Cessna 172 nav and com radio:EN11-HSM1BF20, F.Cu at (192.7, 52.7)
- added U5: MAX7219 COM standby, Package_SO:SSOP-24_3.9x8.7mm_P0.635mm, B.Cu at (135.1, 32.5)
- added U6: 3651A, Cessna 172 nav and com radio:3651A, F.Cu at (135.1, 32.5)
- added U7: MAX7219 COM standby, Package_SO:SSOP-24_3.9x8.7mm_P0.635mm, B.Cu at (178.2, 32.5)
- added U8: 3651A, Cessna 172 nav and com radio:3651A, F.Cu at (178.2, 32.5)
- D1: footprint LED_THT:LED_D5.0mm -> LED_SMD:LED_0805_2012Metric_Pad1.15x1.40mm_HandSolder
- D2: footprint LED_SMD:LED_0805_2012Metric_Pad1.15x1.40mm_HandSolder -> LED_THT:LED_D5.0mm
- J2: value Conn_01x05 -> Barrel_Jack_MountingPin; footprint Connector_PinHeader_2.54mm:PinHeader_1x05_P2.54mm_Vertical -> Cessna 172 nav and com radio:BarrelJack_Horizontal
- J3: value Barrel_Jack_MountingPin -> Conn_01x05; footprint Cessna 172 nav and com radio:BarrelJack_Horizontal -> Connector_PinHeader_2.54mm:PinHeader_1x05_P2.54mm_Vertical
- R2: moved to B.Cu
- SW1: value COMM toggle -> SW_Push; footprint Cessna 172 nav and com radio:B3W-9000-xxx -> Button_Switch_THT:SW_PUSH-12mm
- SW2: value NAV toggle -> SW_Push; footprint Cessna 172 nav and com radio:B3W-9000-xxx -> Button_Switch_THT:SW_PUSH-12mm
- SW3: value Tuning encoder -> SW_Push; footprint Cessna 172 nav and com radio:EN11-HSM1BF20 -> Button_Switch_THT:SW_PUSH-12mm
- SW6: value Ident switch -> Tuning encoder; footprint Cessna 172 nav and com radio:B3W-9000-xxx -> Cessna 172 nav and com radio:EN11-HSM1BF20
- U2, U4: value MAX7219 COM standby -> 3651A; footprint Package_SO:SSOP-24_3.9x8.7mm_P0.635mm -> Cessna 172 nav and com radio:3651A; moved to F.Cu
- moved SW4 251.0 mm to (36.0, 60.7)
- moved J2 162.1 mm to (28.4, 34.8), turned to 0 degrees
- moved SW6 159.0 mm to (104.1, 52.7)
- moved U4 152.9 mm to (89.6, 32.5), turned to 0 degrees
- moved C7 126.9 mm to (31.7, 79.9), turned to 0 degrees
- moved RV1 123.2 mm to (115.4, 51.1)
- moved R1 123.2 mm to (129.7, 58.2)
- moved R8 123.1 mm to (31.7, 74.0), turned to 0 degrees
- moved R6 120.8 mm to (41.2, 74.0), turned to 0 degrees
- moved R7 113.4 mm to (36.5, 74.0), turned to 0 degrees
- moved R5 111.1 mm to (31.7, 77.0), turned to 0 degrees
- moved C6 109.9 mm to (36.5, 77.0), turned to 0 degrees
- moved R10 104.1 mm to (192.7, 67.7), turned to 0 degrees
- moved R12 101.6 mm to (187.9, 70.7), turned to 0 degrees
- moved C9 100.9 mm to (192.7, 64.8), turned to 0 degrees
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Connections:
- J1 pad 13: NAV_TX_LED -> COMM_VOL_LEFT
- J1 pad 15: COMM_VOL_LEFT -> COMM_VOL_RIGHT
- J1 pad 16: COMM_TX_LED -> TEST_SW
- J1 pad 17: COMM_VOL_RIGHT -> IDENT_SW
- J1 pad 18: TEST_SW -> TEST_LED
- J1 pad 19: IDENT_SW -> IDENT_LED
- J1 pad 20: TEST_LED -> Net-(J1-Pad20)
- J1 pad 21: IDENT_LED -> Net-(J1-Pad21)
- R14 pad 1: +5V -> /sheet5F5E0D6C/B
- R14 pad 2: /sheet5F5E0D6C/A -> +5V
- R15 pad 1: /sheet5F5E0D6C/B -> COMM_VOL_LEFT
- R15 pad 2: +5V -> /sheet5F5E0D6C/A
- R16 pad 1: COMM_VOL_LEFT -> /sheet5F5E0D6C/B
- R16 pad 2: /sheet5F5E0D6C/A -> COMM_VOL_RIGHT
- R2 pad 2: TEST_LED -> +5V
- R3 pad 2: +5V -> TEST_LED
- SW1 pad 1: Net-(SW1-Pad1) -> GND
- SW1 pad 2: Net-(SW1-Pad2) -> COMM_TX_SW
- SW2 pad 1: Net-(SW2-Pad1) -> GND
- SW2 pad 2: Net-(SW2-Pad2) -> NAV_TX_SW
- SW4 pad A: /sheet5F5DD32A/A -> /Tuning rotary encoder and switch/A
- SW4 pad B: /sheet5F5DD32A/B -> /Tuning rotary encoder and switch/B
- SW4 pad S1: NAV_KHZ_SW -> COMM_KHZ_SW
- U2 pad 1: /sheet5F611637/DIN -> /5 digit LCD display/SEG_E
- U2 pad 10: Net-(U2-Pad10) -> /5 digit LCD display/DIG_2
- U2 pad 11: /sheet5F611637/DIG_1 -> /5 digit LCD display/DIG_1
- U2 pad 12: LOAD -> /5 digit LCD display/SEG_F
- U2 pad 13: CLK -> /5 digit LCD display/SEG_A
- U2 pad 14: /sheet5F611637/SEG_A -> /5 digit LCD display/DIG_0
- U2 pad 2: /sheet5F611637/DIG_0 -> /5 digit LCD display/SEG_D
- U2 pad 3: /sheet5F611637/DIG_4 -> /5 digit LCD display/SEG_DP
- U2 pad 4: GND -> /5 digit LCD display/SEG_C
- U2 pad 5: Net-(U2-Pad5) -> /5 digit LCD display/SEG_G
- U2 pad 6: /sheet5F611637/DIG_2 -> /5 digit LCD display/DIG_3
- U2 pad 7: /sheet5F611637/DIG_3 -> (no net)
- U2 pad 8: Net-(U2-Pad8) -> /5 digit LCD display/DIG_4
- U2 pad 9: GND -> /5 digit LCD display/SEG_B
- U3 pad 1: /sheet5F613960/DIN -> /sheet5F611637/DIN
- U3 pad 11: /sheet5F613960/DIG_1 -> /sheet5F611637/DIG_1
- U3 pad 14: /sheet5F613960/SEG_A -> /sheet5F611637/SEG_A
- U3 pad 15: /sheet5F613960/SEG_F -> /sheet5F611637/SEG_F
- U3 pad 16: /sheet5F613960/SEG_B -> /sheet5F611637/SEG_B
- U3 pad 17: /sheet5F613960/SEG_G -> /sheet5F611637/SEG_G
- U3 pad 2: /sheet5F613960/DIG_0 -> /sheet5F611637/DIG_0
- U3 pad 20: /sheet5F613960/SEG_C -> /sheet5F611637/SEG_C
- U3 pad 21: /sheet5F613960/SEG_E -> /sheet5F611637/SEG_E
- U3 pad 22: /sheet5F613960/SEG_DP -> /sheet5F611637/SEG_DP
- U3 pad 23: /sheet5F613960/SEG_D -> /sheet5F611637/SEG_D
- U3 pad 24: /sheet5F613961/DIN -> /sheet5F613960/DIN
- U3 pad 3: /sheet5F613960/DIG_4 -> /sheet5F611637/DIG_4
- U3 pad 6: /sheet5F613960/DIG_2 -> /sheet5F611637/DIG_2
- U3 pad 7: /sheet5F613960/DIG_3 -> /sheet5F611637/DIG_3
- U4 pad 1: /sheet5F613961/DIN -> /sheet5F611637/SEG_E
- U4 pad 10: Net-(U4-Pad10) -> /sheet5F611637/DIG_2
- U4 pad 11: /sheet5F613961/DIG_1 -> /sheet5F611637/DIG_1
- U4 pad 12: LOAD -> /sheet5F611637/SEG_F
- U4 pad 13: CLK -> /sheet5F611637/SEG_A
- U4 pad 14: /sheet5F613961/SEG_A -> /sheet5F611637/DIG_0
- U4 pad 2: /sheet5F613961/DIG_0 -> /sheet5F611637/SEG_D
- U4 pad 3: /sheet5F613961/DIG_4 -> /sheet5F611637/SEG_DP
- U4 pad 4: GND -> /sheet5F611637/SEG_C
- U4 pad 5: Net-(U4-Pad5) -> /sheet5F611637/SEG_G
- U4 pad 6: /sheet5F613961/DIG_2 -> /sheet5F611637/DIG_3
- U4 pad 7: /sheet5F613961/DIG_3 -> (no net)
- U4 pad 8: Net-(U4-Pad8) -> /sheet5F611637/DIG_4
- U4 pad 9: GND -> /sheet5F611637/SEG_B
Routing:
- net (no net): track 0.00 -> 150.0 mm, vias 0 -> 1
- net /sheet5F613961/SEG_D: track 115.0 -> 0.00 mm, vias 5 -> 0
- net /sheet5F611637/SEG_D: track 115.0 -> 3.75 mm, vias 5 -> 0
- net /5 digit LCD display/SEG_D: track 115.0 -> 3.75 mm, vias 5 -> 0
- net /sheet5F613960/SEG_D: track 115.0 -> 3.75 mm, vias 5 -> 0
- net /sheet5F613961/SEG_DP: track 105.0 -> 0.00 mm, vias 1 -> 0
- net /sheet5F613961/SEG_E: track 105.8 -> 1.14 mm, vias 5 -> 1
- net /5 digit LCD display/SEG_DP: track 105.0 -> 2.61 mm, vias 1 -> 0
- net /sheet5F611637/SEG_DP: track 105.0 -> 2.61 mm, vias 1 -> 0
- net /sheet5F613960/SEG_DP: track 105.0 -> 2.61 mm, vias 1 -> 0
- net /sheet5F613961/SEG_C: track 95.8 -> 0.00 mm, vias 6 -> 0
- net /sheet5F613960/SEG_E: track 105.8 -> 10.8 mm, vias 5 -> 0
- net /5 digit LCD display/SEG_E: track 105.8 -> 10.8 mm, vias 5 -> 0
- net /sheet5F611637/SEG_E: track 105.8 -> 10.8 mm, vias 5 -> 0
- net /5 digit LCD display/SEG_C: track 95.8 -> 2.87 mm, vias 6 -> 0
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Other:
- board size 289 x 69 mm -> 187.7 x 71.1 mm
- board text removed: "COMM encoder"
- board text removed: "COMM test LED"
- board text removed: "COMM volume encoder"
- board text removed: "NAV encoder"

Commit message: New board size!
Parts:
- added REF**: MountingHole_3mm, MountingHole:MountingHole_3mm, F.Cu at (205.0, 125.0)
- added REF**: MountingHole_3mm, MountingHole:MountingHole_3mm, F.Cu at (205.0, 153.0)
- added REF**: MountingHole_3mm, MountingHole:MountingHole_3mm, F.Cu at (35.0, 153.0)
- added REF**: MountingHole_3mm, MountingHole:MountingHole_3mm, F.Cu at (35.0, 125.0)
- C10, C11, C6, C7, C8, C9, D1, R10, R11, R12, R13, R14, R15, R16, R5, R6, R7, R8, R9: moved to B.Cu
- D2: moved to F.Cu
- SW1, SW2, SW3: footprint Button_Switch_THT:SW_PUSH-12mm -> Button_Switch_THT:SW_PUSH_6mm_H8mm
- moved J1 162.0 mm to (150.0, 143.5), turned to 90 degrees
- moved C1 128.9 mm to (44.0, 147.8), turned to 0 degrees
- moved R2 119.6 mm to (44.0, 154.0), turned to 90 degrees
- moved J3 119.3 mm to (163.0, 155.0)
- moved D3 114.6 mm to (138.5, 152.5)
- moved SW4 110.8 mm to (38.5, 171.5)
- moved R1 109.3 mm to (66.2, 147.2)
- moved RV1 109.3 mm to (51.9, 140.1)
- moved R8 109.3 mm to (41.0, 183.0), turned to 270 degrees
- moved R6 109.1 mm to (47.0, 183.0), turned to 270 degrees
- moved R7 109.0 mm to (36.0, 183.0), turned to 90 degrees
- moved C6 106.1 mm to (33.0, 183.0), turned to 90 degrees
- moved R5 106.0 mm to (30.0, 183.0), turned to 90 degrees
- moved J2 105.4 mm to (44.0, 139.0)
- moved C7 103.8 mm to (44.0, 183.0), turned to 270 degrees
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Routing:
- net (no net): track 150.0 -> 0.00 mm, vias 1 -> 0
- net /sheet5F613961/SEG_A: track 0.00 -> 31.4 mm
- net /sheet5F613961/SEG_F: track 0.00 -> 27.9 mm
- net /sheet5F613961/SEG_B: track 1.15 -> 19.3 mm, vias 1 -> 0
- net /sheet5F613961/DIG_4: track 0.00 -> 16.9 mm
- net GND: track 22.9 -> 36.1 mm, vias 12 -> 17
- net /sheet5F613961/SEG_E: track 1.14 -> 10.8 mm, vias 1 -> 0
- net /Tuning rotary encoder and switch/B: track 0.00 -> 9.09 mm
- net /Tuning rotary encoder and switch/A: track 0.00 -> 9.00 mm
- net /sheet5F613961/DIN: track 14.7 -> 6.10 mm
- net CLK: track 37.1 -> 45.7 mm
- net /sheet5F613961/DIG_1: track 0.00 -> 8.39 mm
- net +5V: track 44.2 -> 37.4 mm
- net /sheet5F613961/DIG_0: track 0.00 -> 6.24 mm
- net /sheet5F613961/DIG_2: track 0.00 -> 4.38 mm
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- removed copper zone on B.Cu, net GND
- removed copper zone on F.Cu, net GND
Other:
- board size 187.7 x 71.1 mm -> 180 x 38 mm
- board text added: "180x38"
- board text added: "IDENT LED"
- board text added: "TEST LED"
