File: Autopilot panel/rotary encoder.sch (KiCad schematic (older format))
At the start: 7 parts

Commit message: New board ready
Parts:
- C2, C3: renamed from C?; footprint (none) -> Capacitor_SMD:C_0805_2012Metric_Pad1.15x1.40mm_HandSolder; LCSC (none) -> C1710
- J3: renamed from J?; footprint EN11HSM1BF20 -> SamacSys_Parts:EN11HSM1BF20
- R6, R7: renamed from R?; footprint (none) -> Resistor_SMD:R_0805_2012Metric_Pad1.15x1.40mm_HandSolder; LCSC (none) -> C17414
- R8, R9: renamed from R?; value R -> 10k; footprint (none) -> Resistor_SMD:R_0805_2012Metric_Pad1.15x1.40mm_HandSolder; LCSC (none) -> C17414
Connections:
- net +5V: now also R6.1, R7.1; no longer R6.2, R7.2
- net RIGHT: now also R9.1; no longer R9.2
- net A1: now reaches C2.2, J3.A1, R8.2
- net A1: now also R6.2; no longer R6.1
- net B1: now reaches C3.2, J3.B1
- net B1: now also R7.2, R9.2; no longer R7.1, R9.1

Commit message: more autopilot changes
Changed lines of the file:
@@
 $Descr A4 11693 8268
 encoding utf-8
-Sheet 6 6
+Sheet 2 6
 Title ""
 Date ""
@@
 AR Path="/5F811ACB/5F810CE8" Ref="J6"  Part="1"
 AR Path="/5F811C24/5F810CE8" Ref="J7"  Part="1"
-F 0 "J7" V 5519 2650 50  0000 C CNN
+F 0 "J3" V 5519 2650 50  0000 C CNN
 F 1 "EN11-HSM1BF20" V 5610 2650 50  0000 C CNN
 F 2 "SamacSys_Parts:EN11HSM1BF20" H 6550 2950 50  0001 L CNN
@@
 AR Path="/5F811ACB/5F810CFC" Ref="R18"  Part="1"
 AR Path="/5F811C24/5F810CFC" Ref="R22"  Part="1"
-F 0 "R22" V 4593 3050 50  0000 C CNN
+F 0 "R6" V 4593 3050 50  0000 C CNN
 F 1 "10k" V 4684 3050 50  0000 C CNN
 F 2 "Resistor_SMD:R_0805_2012Metric_Pad1.15x1.40mm_HandSolder" V 4730 3050 50  0001 C CNN
@@
 AR Path="/5F811ACB/5F810D02" Ref="R19"  Part="1"
 AR Path="/5F811C24/5F810D02" Ref="R23"  Part="1"
-F 0 "R23" V 4900 3250 50  0000 C CNN
+F 0 "R7" V 4900 3250 50  0000 C CNN
 F 1 "10k" V 5000 3250 50  0000 C CNN
 F 2 "Resistor_SMD:R_0805_2012Metric_Pad1.15x1.40mm_HandSolder" V 4730 3250 50  0001 C CNN
@@
 AR Path="/5F811ACB/5F810D13" Ref="C9"  Part="1"
 AR Path="/5F811C24/5F810D13" Ref="C11"  Part="1"
-F 0 "C11" V 5298 3950 50  0000 C CNN
+F 0 "C3" V 5298 3950 50  0000 C CNN
 F 1 "0.01uf" V 5389 3950 50  0000 C CNN
 F 2 "Capacitor_SMD:C_0805_2012Metric_Pad1.15x1.40mm_HandSolder" H 5588 3800 50  0001 C CNN
@@
 AR Path="/5F811ACB/5F810D19" Ref="C8"  Part="1"
 AR Path="/5F811C24/5F810D19" Ref="C10"  Part="1"
-F 0 "C10" V 5298 2300 50  0000 C CNN
+F 0 "C2" V 5298 2300 50  0000 C CNN
 F 1 "0.01uF" V 5389 2300 50  0000 C CNN
 F 2 "Capacitor_SMD:C_0805_2012Metric_Pad1.15x1.40mm_HandSolder" H 5588 2150 50  0001 C CNN
@@
 AR Path="/5F811ACB/5F810D33" Ref="R21"  Part="1"
 AR Path="/5F811C24/5F810D33" Ref="R25"  Part="1"
-F 0 "R25" H 5170 4146 50  0000 L CNN
+F 0 "R9" H 5170 4146 50  0000 L CNN
 F 1 "10k" H 5170 4055 50  0000 L CNN
 F 2 "Resistor_SMD:R_0805_2012Metric_Pad1.15x1.40mm_HandSolder" V 5030 4100 50  0001 C CNN
@@
 AR Path="/5F811ACB/5F810D3A" Ref="R20"  Part="1"
 AR Path="/5F811C24/5F810D3A" Ref="R24"  Part="1"
-F 0 "R24" H 5170 2196 50  0000 L CNN
+F 0 "R8" H 5170 2196 50  0000 L CNN
 F 1 "10k" H 5170 2105 50  0000 L CNN
 F 2 "Resistor_SMD:R_0805_2012Metric_Pad1.15x1.40mm_HandSolder" V 5030 2150 50  0001 C CNN
