File: Autopilot panel/Autopilot panel.kicad_pcb (KiCad board)
At the start: 2 copper layers, 133 x 58 mm, 59 parts, among them J1 USB_B_Micro, J2 Conn_02x15_Odd_Even, J3 EN11-HSM1BF20, J4 EN11-HSM1BF20, J5 EN11-HSM1BF20, J6 EN11-HSM1BF20, J7 EN11-HSM1BF20, SW1 SW_Push, SW2 SW_Push, SW3 SW_Push, SW4 SW_Push, SW5 SW_Push

Commit message: more autopilot changes
Parts:
- added J8: Conn_02x15_Odd_Even, Connector_PinHeader_2.54mm:PinHeader_2x15_P2.54mm_Vertical, B.Cu at (97.8, 66.0)
- D1, D2, D3, D4, D5: value LED -> LED_RCBG; footprint LED_THT:LED_D5.0mm -> LED_THT:LED_D5.0mm-4_RGB
- J2: footprint Connector_PinSocket_2.54mm:PinSocket_2x15_P2.54mm_Vertical -> Connector_PinHeader_2.54mm:PinHeader_2x15_P2.54mm_Vertical
- moved J2 3.01 mm to (97.8, 115.0)
- moved R1 1.12 mm to (68.5, 74.0)
- moved R2 1.12 mm to (94.5, 74.0)
- moved R3 1.12 mm to (120.5, 74.0)
- moved R4 1.12 mm to (146.5, 74.0)
- moved D5 1.00 mm to (166.0, 73.0)
- moved R5 1.00 mm to (173.0, 73.0)
- moved D1 0.50 mm to (61.5, 74.0)
- moved D2 0.50 mm to (87.5, 74.0)
- moved D3 0.50 mm to (113.5, 74.0)
- moved D4 0.50 mm to (139.5, 74.0)
Connections:
- D1 pad 1: GND -> LED1_R
- D2 pad 1: GND -> LED2_R
- D3 pad 1: GND -> LED3_R
- D4 pad 1: GND -> LED4_R
- D5 pad 1: GND -> LED5_R
- J2 pad 1: LED1 -> ENC1_SW
- J2 pad 10: ENC1_RIGHT -> Net-(J2-Pad10)
- J2 pad 11: SW1 -> ENC2_RIGHT
- J2 pad 12: ENC2_SW -> Net-(J2-Pad12)
- J2 pad 13: SW2 -> ENC3_SW
- J2 pad 14: ENC2_LEFT -> Net-(J2-Pad14)
- J2 pad 15: SW3 -> ENC3_LEFT
- J2 pad 16: ENC2_RIGHT -> Net-(J2-Pad16)
- J2 pad 17: SW4 -> ENC3_RIGHT
- J2 pad 18: ENC3_SW -> Net-(J2-Pad18)
- J2 pad 19: SW5 -> ENC4_SW
- J2 pad 20: ENC3_LEFT -> Net-(J2-Pad20)
- J2 pad 21: ENC5_SW -> ENC4_LEFT
- J2 pad 22: ENC3_RIGHT -> Net-(J2-Pad22)
- J2 pad 23: ENC5_LEFT -> ENC4_RIGHT
- J2 pad 24: ENC4_SW -> Net-(J2-Pad24)
- J2 pad 26: ENC4_LEFT -> Net-(J2-Pad26)
- J2 pad 27: GND -> ENC5_LEFT
- J2 pad 28: ENC4_RIGHT -> Net-(J2-Pad28)
- J2 pad 29: GND -> ENC5_SW
- J2 pad 3: LED2 -> ENC1_LEFT
- J2 pad 30: GND -> Net-(J2-Pad30)
- J2 pad 5: LED3 -> ENC1_RIGHT
- J2 pad 6: ENC1_SW -> Net-(J2-Pad6)
- J2 pad 7: LED4 -> ENC2_SW
- J2 pad 8: ENC1_LEFT -> Net-(J2-Pad8)
- J2 pad 9: LED5 -> ENC2_LEFT
- R1 pad 1: LED1 -> Net-(D1-Pad2)
- R1 pad 2: Net-(D1-Pad2) -> GND
- R2 pad 1: LED2 -> Net-(D2-Pad2)
- R2 pad 2: Net-(D2-Pad2) -> GND
- R3 pad 1: LED3 -> Net-(D3-Pad2)
- R3 pad 2: Net-(D3-Pad2) -> GND
- R4 pad 1: LED4 -> Net-(D4-Pad2)
- R4 pad 2: Net-(D4-Pad2) -> GND
- R5 pad 1: LED5 -> Net-(D5-Pad2)
- R5 pad 2: Net-(D5-Pad2) -> GND
Routing:
- net LED5: track 113.9 -> 0.00 mm
- net LED4: track 74.7 -> 0.00 mm, vias 1 -> 0
- net LED2: track 68.3 -> 0.00 mm, vias 1 -> 0
- net LED1: track 59.2 -> 0.00 mm, vias 2 -> 0
- net LED3: track 52.7 -> 0.00 mm, vias 1 -> 0
- net LED1_B: track 0.00 -> 46.0 mm
- net LED5_G: track 0.00 -> 42.8 mm
- net LED5_R: track 0.00 -> 40.6 mm
- net LED1_R: track 0.00 -> 39.2 mm
- net LED1_G: track 0.00 -> 38.2 mm
- net LED5_B: track 0.00 -> 37.8 mm
- net LED2_B: track 0.00 -> 23.6 mm
- net LED4_G: track 0.00 -> 23.4 mm
- net SW1: track 68.2 -> 45.8 mm
- net LED4_R: track 0.00 -> 21.4 mm
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
Commit message: Submitted version!
Parts:
- removed R1, R2, R3, R4, R5: 220, Resistor_SMD:R_0805_2012Metric_Pad1.15x1.40mm_HandSolder
- added RN1: 470, Resistor_SMD:R_Array_Convex_4x0603, F.Cu at (56.5, 74.0)
- added RN2: 470, Resistor_SMD:R_Array_Convex_4x0603, F.Cu at (89.0, 74.5)
- added RN3: 470, Resistor_SMD:R_Array_Convex_4x0603, F.Cu at (121.0, 74.5)
- added RN4: 470, Resistor_SMD:R_Array_Convex_4x0603, F.Cu at (153.0, 74.0)
- added RN5: 470, Resistor_SMD:R_Array_Convex_4x0603, F.Cu at (185.5, 73.0)
- C1: footprint Capacitor_Tantalum_SMD:CP_EIA-3216-18_Kemet-A -> Capacitor_THT:CP_Radial_D5.0mm_P2.00mm; moved to B.Cu
- moved D6 22.1 mm to (42.5, 89.0), turned to 180 degrees
- moved R26 17.9 mm to (42.5, 86.0), turned to 0 degrees
- moved J1 16.5 mm to (35.7, 86.0)
- moved C1 15.4 mm to (41.6, 80.3)
- moved HOLE1 15.0 mm to (39.0, 69.0)
- moved HOLE2 15.0 mm to (39.0, 115.0)
- moved HOLE3 15.0 mm to (192.0, 115.0)
- moved HOLE4 15.0 mm to (192.0, 69.0)
- moved D5 14.1 mm to (180.0, 75.0), turned to 90 degrees
- moved C10 12.4 mm to (169.0, 108.0)
- moved C11 12.4 mm to (190.0, 108.0)
- moved C2 12.4 mm to (41.0, 108.0)
- moved C3 12.4 mm to (62.0, 108.0)
- moved J3 12.4 mm to (49.0, 108.0)
- moved J7 12.4 mm to (177.0, 108.0)
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Connections:
- D1 pad 1: LED1_R -> Net-(D1-Pad1)
- D1 pad 2: Net-(D1-Pad2) -> GND
- D1 pad 3: LED1_B -> Net-(D1-Pad3)
- D1 pad 4: LED1_G -> Net-(D1-Pad4)
- D2 pad 1: LED2_R -> Net-(D2-Pad1)
- D2 pad 2: Net-(D2-Pad2) -> GND
- D2 pad 3: LED2_B -> Net-(D2-Pad3)
- D2 pad 4: LED2_G -> Net-(D2-Pad4)
- D3 pad 1: LED3_R -> Net-(D3-Pad1)
- D3 pad 2: Net-(D3-Pad2) -> GND
- D3 pad 3: LED3_B -> Net-(D3-Pad3)
- D3 pad 4: LED3_G -> Net-(D3-Pad4)
- D4 pad 1: LED4_R -> Net-(D4-Pad1)
- D4 pad 2: Net-(D4-Pad2) -> GND
- D4 pad 3: LED4_B -> Net-(D4-Pad3)
- D4 pad 4: LED4_G -> Net-(D4-Pad4)
- D5 pad 1: LED5_R -> Net-(D5-Pad1)
- D5 pad 2: Net-(D5-Pad2) -> GND
- D5 pad 3: LED5_B -> Net-(D5-Pad3)
- D5 pad 4: LED5_G -> Net-(D5-Pad4)
Routing:
- net LED4_B: track 19.5 -> 67.4 mm
- net LED5_G: track 42.8 -> 63.3 mm
- net LED5_R: track 40.6 -> 60.8 mm
- net LED5_B: track 37.8 -> 57.7 mm
- net +5V: track 226.8 -> 245.4 mm
- net LED4_R: track 21.4 -> 35.3 mm
- net SW5: track 45.3 -> 57.7 mm
- net SW1: track 45.8 -> 58.2 mm
- net Net-(D5-Pad1): track 0.00 -> 12.0 mm
- net LED4_G: track 23.4 -> 35.0 mm
- net ENC1_SW: track 46.9 -> 57.7 mm, vias 1 -> 0
- net ENC5_SW: track 41.8 -> 52.6 mm
- net ENC5_LEFT: track 33.3 -> 43.6 mm
- net ENC1_RIGHT: track 35.9 -> 46.2 mm
- net ENC5_RIGHT: track 66.3 -> 75.6 mm
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Other:
- board size 133 x 58 mm -> 165 x 58 mm
- board text added: "SW1"
