File: Autopilot panel/Autopilot panel.sch (KiCad schematic (older format))
At the start: 17 parts

Commit message: New board ready
Parts:
- added D6: LED, LED_SMD:LED_0805_2012Metric_Pad1.15x1.40mm_HandSolder, symbol Device:LED
- added J2: Conn_02x15_Odd_Even, Connector_PinSocket_2.54mm:PinSocket_2x15_P2.54mm_Vertical, symbol Connector_Generic:Conn_02x15_Odd_Even
- added R26: 220, Resistor_SMD:R_0805_2012Metric_Pad1.15x1.40mm_HandSolder, symbol Device:R
- C1: renamed from C?; footprint (none) -> Capacitor_Tantalum_SMD:CP_EIA-3216-18_Kemet-A; LCSC (none) -> C7171
- D1, D2, D3, D4, D5: renamed from D?; footprint (none) -> LED_THT:LED_D5.0mm
- J1: renamed from J?; footprint (none) -> Connector_USB:USB_Micro-B_Molex-105017-0001
- R1, R2, R3, R4, R5: renamed from R?; value R -> 220; footprint (none) -> Resistor_SMD:R_0805_2012Metric_Pad1.15x1.40mm_HandSolder; LCSC (none) -> C17557
- SW1, SW2, SW3, SW4, SW5: renamed from SW?; footprint (none) -> Button_Switch_THT:SW_PUSH_6mm_H8mm
Connections:
- net +5V: now also J2.2 (Pin_2), R26.1
- net ENC1_LEFT: now also J2.8 (Pin_8)
- net ENC1_RIGHT: now also J2.10 (Pin_10)
- net ENC1_SW: now also J2.6 (Pin_6)
- net ENC2_LEFT: now also J2.14 (Pin_14)
- net ENC2_RIGHT: now also J2.16 (Pin_16)
- net ENC2_SW: now also J2.12 (Pin_12)
- net ENC3_LEFT: now also J2.20 (Pin_20)
- net ENC3_RIGHT: now also J2.22 (Pin_22)
- net ENC3_SW: now also J2.18 (Pin_18)
- net ENC4_LEFT: now also J2.26 (Pin_26)
- net ENC4_RIGHT: now also J2.28 (Pin_28)
- net ENC4_SW: now also J2.24 (Pin_24)
- net ENC5_LEFT: now also J2.23 (Pin_23)
- net ENC5_RIGHT: now also J2.25 (Pin_25)
- net ENC5_SW: now also J2.21 (Pin_21)
- net GND: now also D6.1 (K), J2.27 (Pin_27), J2.29 (Pin_29), J2.30 (Pin_30), J2.4 (Pin_4)
- net LED1: now also J2.1 (Pin_1)
- net LED2: now also J2.3 (Pin_3)
- net LED3: now also J2.5 (Pin_5)
- net LED4: now also J2.7 (Pin_7)
- net LED5: now also J2.9 (Pin_9)
- net SW1: now also J2.11 (Pin_11)
- net SW2: now also J2.13 (Pin_13)
- net SW3: now also J2.15 (Pin_15)
- net SW4: now also J2.17 (Pin_17)
- net SW5: now also J2.19 (Pin_19)
- new net: D6.2 (A), R26.2

Commit message: more autopilot changes
Parts:
- removed D1, D2, D3, D4, D5: LED, LED_THT:LED_D5.0mm, symbol Device:LED
- added D1, D2, D3, D4, D5: LED_RCBG, LED_THT:LED_D5.0mm-4_RGB, symbol Device:LED_RCBG
- added J8: Conn_02x15_Odd_Even, Connector_PinHeader_2.54mm:PinHeader_2x15_P2.54mm_Vertical, symbol Connector_Generic:Conn_02x15_Odd_Even
- J2: footprint Connector_PinSocket_2.54mm:PinSocket_2x15_P2.54mm_Vertical -> Connector_PinHeader_2.54mm:PinHeader_2x15_P2.54mm_Vertical
Connections:
- net ENC1_LEFT: now also J2.3 (Pin_3); no longer J2.8 (Pin_8)
- net ENC1_RIGHT: now also J2.5 (Pin_5); no longer J2.10 (Pin_10)
- net ENC1_SW: now also J2.1 (Pin_1); no longer J2.6 (Pin_6)
- net ENC2_LEFT: now also J2.9 (Pin_9); no longer J2.14 (Pin_14)
- net ENC2_RIGHT: now also J2.11 (Pin_11); no longer J2.16 (Pin_16)
- net ENC2_SW: now also J2.7 (Pin_7); no longer J2.12 (Pin_12)
- net ENC3_LEFT: now also J2.15 (Pin_15); no longer J2.20 (Pin_20)
- net ENC3_RIGHT: now also J2.17 (Pin_17); no longer J2.22 (Pin_22)
- net ENC3_SW: now also J2.13 (Pin_13); no longer J2.18 (Pin_18)
- net ENC4_LEFT: now also J2.21 (Pin_21); no longer J2.26 (Pin_26)
- net ENC4_RIGHT: now also J2.23 (Pin_23); no longer J2.28 (Pin_28)
- net ENC4_SW: now also J2.19 (Pin_19); no longer J2.24 (Pin_24)
- net ENC5_LEFT: now also J2.27 (Pin_27); no longer J2.23 (Pin_23)
- net ENC5_SW: now also J2.29 (Pin_29); no longer J2.21 (Pin_21)
- net GND: now also R1.2, R2.2, R3.2, R4.2, R5.2; no longer J2.27 (Pin_27), J2.29 (Pin_29), J2.30 (Pin_30)
- net SW1: now also J8.1 (Pin_1); no longer J2.11 (Pin_11)
- net SW2: now also J8.9 (Pin_9); no longer J2.13 (Pin_13)
- net SW3: now also J8.15 (Pin_15); no longer J2.15 (Pin_15)
- net SW4: now also J8.21 (Pin_21); no longer J2.17 (Pin_17)
- net SW5: now also J8.29 (Pin_29); no longer J2.19 (Pin_19)
- net LED1: no longer names the net of R1.1
- net LED1: now also D1.2 (K); no longer J2.1 (Pin_1)
- net LED2: no longer names the net of R2.1
- net LED2: now also D2.2 (K); no longer J2.3 (Pin_3)
- net LED3: no longer names the net of R3.1
- net LED3: now also D3.2 (K); no longer J2.5 (Pin_5)
- net LED4: no longer names the net of R4.1
- net LED4: now also D4.2 (K); no longer J2.7 (Pin_7)
- net LED5: no longer names the net of R5.1
- net LED5: now also D5.2 (K); no longer J2.9 (Pin_9)
- new net LED1_B: D1.3 (BA), J8.6 (Pin_6)
- new net LED1_G: D1.4 (GA), J8.4 (Pin_4)
- new net LED1_R: D1.1 (RA), J8.2 (Pin_2)
- new net LED2_B: D2.3 (BA), J8.12 (Pin_12)
- new net LED2_G: D2.4 (GA), J8.10 (Pin_10)
- new net LED2_R: D2.1 (RA), J8.8 (Pin_8)
- new net LED3_B: D3.3 (BA), J8.18 (Pin_18)
- new net LED3_G: D3.4 (GA), J8.16 (Pin_16)
- new net LED3_R: D3.1 (RA), J8.14 (Pin_14)
- new net LED4_B: D4.3 (BA), J8.24 (Pin_24)
- new net LED4_G: D4.4 (GA), J8.22 (Pin_22)
- new net LED4_R: D4.1 (RA), J8.20 (Pin_20)
- new net LED5_B: D5.3 (BA), J8.30 (Pin_30)
- new net LED5_G: D5.4 (GA), J8.28 (Pin_28)
- new net LED5_R: D5.1 (RA), J8.26 (Pin_26)
- no-connect marks 4 -> 27
Other:
- moved on the sheet: R1

Commit message: Submitted version!
Parts:
- removed R1, R2, R3, R4, R5: 220, Resistor_SMD:R_0805_2012Metric_Pad1.15x1.40mm_HandSolder, symbol Device:R
- added RN1, RN2, RN3, RN4, RN5: 470, Resistor_SMD:R_Array_Convex_4x0603, symbol Device:R_Pack04
- C1: footprint Capacitor_Tantalum_SMD:CP_EIA-3216-18_Kemet-A -> Capacitor_THT:CP_Radial_D5.0mm_P2.00mm
Connections:
- net GND: now also D1.2 (K), D2.2 (K), D3.2 (K), D4.2 (K), D5.2 (K)
- net LED1_B: now also RN1.6 (R3.2); no longer D1.3 (BA)
- net LED1_G: now also RN1.7 (R2.2); no longer D1.4 (GA)
- net LED1_R: now also RN1.8 (R1.2); no longer D1.1 (RA)
- net LED2_B: now also RN2.6 (R3.2); no longer D2.3 (BA)
- net LED2_G: now also RN2.7 (R2.2); no longer D2.4 (GA)
- net LED2_R: now also RN2.8 (R1.2); no longer D2.1 (RA)
- net LED3_B: now also RN3.6 (R3.2); no longer D3.3 (BA)
- net LED3_G: now also RN3.7 (R2.2); no longer D3.4 (GA)
- net LED3_R: now also RN3.8 (R1.2); no longer D3.1 (RA)
- net LED4_B: now also RN4.6 (R3.2); no longer D4.3 (BA)
- net LED4_G: now also RN4.7 (R2.2); no longer D4.4 (GA)
- net LED4_R: now also RN4.8 (R1.2); no longer D4.1 (RA)
- net LED5_B: now also RN5.6 (R3.2); no longer D5.3 (BA)
- net LED5_G: now also RN5.7 (R2.2); no longer D5.4 (GA)
- net LED5_R: now also RN5.8 (R1.2); no longer D5.1 (RA)
- new net: D1.1 (RA), RN1.1 (R1.1)
- new net: D1.3 (BA), RN1.3 (R3.1)
- new net: D1.4 (GA), RN1.2 (R2.1)
- new net: D2.1 (RA), RN2.1 (R1.1)
- new net: D2.3 (BA), RN2.3 (R3.1)
- new net: D2.4 (GA), RN2.2 (R2.1)
- new net: D3.1 (RA), RN3.1 (R1.1)
- new net: D3.3 (BA), RN3.3 (R3.1)
- new net: D3.4 (GA), RN3.2 (R2.1)
- new net: D4.1 (RA), RN4.1 (R1.1)
- new net: D4.3 (BA), RN4.3 (R3.1)
- new net: D4.4 (GA), RN4.2 (R2.1)
- new net: D5.1 (RA), RN5.1 (R1.1)
- new net: D5.3 (BA), RN5.3 (R3.1)
- new net: D5.4 (GA), RN5.2 (R2.1)
- no-connect marks 27 -> 37
