File: USB breakout/USB breakout.sch (KiCad schematic (older format))
At the start: 11 parts, among them J1 USB_B_Micro, J2 Conn_01x06_Female

Commit message: Swap to different USB footprint
Parts:
- J1: footprint Connector_USB:USB_Micro-B_Molex-105017-0001 -> digikey-footprints:USB_Micro_B_Female_10118194-0001LF; symbol Connector:USB_B_Micro -> USB-breakout-rescue:USB_B_Micro-Connector
Changed lines of the file:
@@
 $EndDescr
 $Comp
-L Connector:USB_B_Micro J1
+L USB-breakout-rescue:USB_B_Micro-Connector J1
 U 1 1 6125557F
 P 2100 3300
 F 0 "J1" H 2157 3767 50  0000 C CNN
 F 1 "USB_B_Micro" H 2157 3676 50  0000 C CNN
-F 2 "Connector_USB:USB_Micro-B_Molex-105017-0001" H 2250 3250 50  0001 C CNN
+F 2 "digikey-footprints:USB_Micro_B_Female_10118194-0001LF" H 2250 3250 50  0001 C CNN
 F 3 "~" H 2250 3250 50  0001 C CNN
 	1    2100 3300

Commit message: Upsize all the connectors
Parts:
- C1, C2, C3, C4: footprint Capacitor_SMD:C_0805_2012Metric_Pad1.15x1.40mm_HandSolder -> Capacitor_SMD:C_1206_3216Metric_Pad1.33x1.80mm_HandSolder
- D1: footprint LED_SMD:LED_0805_2012Metric_Pad1.15x1.40mm_HandSolder -> LED_SMD:LED_1206_3216Metric_Pad1.42x1.75mm_HandSolder
- FB1, R1, R2, R3: footprint Resistor_SMD:R_0805_2012Metric_Pad1.15x1.40mm_HandSolder -> Resistor_SMD:R_1206_3216Metric_Pad1.30x1.75mm_HandSolder
- J1: footprint digikey-footprints:USB_Micro_B_Female_10118194-0001LF -> Connector_USB:USB_Micro-B_Amphenol_10118194_Horizontal
Changed lines of the file:
@@
 F 0 "J1" H 2157 3767 50  0000 C CNN
 F 1 "USB_B_Micro" H 2157 3676 50  0000 C CNN
-F 2 "digikey-footprints:USB_Micro_B_Female_10118194-0001LF" H 2250 3250 50  0001 C CNN
+F 2 "Connector_USB:USB_Micro-B_Amphenol_10118194_Horizontal" H 2250 3250 50  0001 C CNN
 F 3 "~" H 2250 3250 50  0001 C CNN
 	1    2100 3300
@@
 F 0 "R1" V 2643 3400 50  0000 C CNN
 F 1 "22" V 2734 3400 50  0000 C CNN
-F 2 "Resistor_SMD:R_0805_2012Metric_Pad1.15x1.40mm_HandSolder" V 2780 3400 50  0001 C CNN
+F 2 "Resistor_SMD:R_1206_3216Metric_Pad1.30x1.75mm_HandSolder" V 2780 3400 50  0001 C CNN
 F 3 "~" H 2850 3400 50  0001 C CNN
 	1    2850 3400
@@
 F 0 "R2" V 2643 3700 50  0000 C CNN
 F 1 "22" V 2734 3700 50  0000 C CNN
-F 2 "Resistor_SMD:R_0805_2012Metric_Pad1.15x1.40mm_HandSolder" V 2780 3700 50  0001 C CNN
+F 2 "Resistor_SMD:R_1206_3216Metric_Pad1.30x1.75mm_HandSolder" V 2780 3700 50  0001 C CNN
 F 3 "~" H 2850 3700 50  0001 C CNN
 	1    2850 3700
@@
 F 0 "D1" V 4739 3433 50  0000 R CNN
 F 1 "LED" V 4648 3433 50  0000 R CNN
-F 2 "LED_SMD:LED_0805_2012Metric_Pad1.15x1.40mm_HandSolder" H 4700 3550 50  0001 C CNN
+F 2 "LED_SMD:LED_1206_3216Metric_Pad1.42x1.75mm_HandSolder" H 4700 3550 50  0001 C CNN
 F 3 "~" H 4700 3550 50  0001 C CNN
 	1    4700 3550
@@
 F 0 "R3" H 4770 3296 50  0000 L CNN
 F 1 "1K" H 4770 3205 50  0000 L CNN
-F 2 "Resistor_SMD:R_0805_2012Metric_Pad1.15x1.40mm_HandSolder" V 4630 3250 50  0001 C CNN
+F 2 "Resistor_SMD:R_1206_3216Metric_Pad1.30x1.75mm_HandSolder" V 4630 3250 50  0001 C CNN
 F 3 "~" H 4700 3250 50  0001 C CNN
 	1    4700 3250
@@
 F 0 "C3" H 4415 3296 50  0000 L CNN
 F 1 "0.1uF" H 4415 3205 50  0000 L CNN
-F 2 "Capacitor_SMD:C_0805_2012Metric_Pad1.15x1.40mm_HandSolder" H 4338 3100 50  0001 C CNN
+F 2 "Capacitor_SMD:C_1206_3216Metric_Pad1.33x1.80mm_HandSolder" H 4338 3100 50  0001 C CNN
 F 3 "~" H 4300 3250 50  0001 C CNN
 	1    4300 3250
@@
 F 0 "C2" H 4015 3296 50  0000 L CNN
 F 1 "1uF" H 4015 3205 50  0000 L CNN
-F 2 "Capacitor_SMD:C_0805_2012Metric_Pad1.15x1.40mm_HandSolder" H 3938 3100 50  0001 C CNN
+F 2 "Capacitor_SMD:C_1206_3216Metric_Pad1.33x1.80mm_HandSolder" H 3938 3100 50  0001 C CNN
 F 3 "~" H 3900 3250 50  0001 C CNN
 	1    3900 3250
@@
 F 0 "C4" V 5298 3750 50  0000 C CNN
 F 1 "1uF" V 5389 3750 50  0000 C CNN
-F 2 "Capacitor_SMD:C_0805_2012Metric_Pad1.15x1.40mm_HandSolder" H 5588 3600 50  0001 C CNN
+F 2 "Capacitor_SMD:C_1206_3216Metric_Pad1.33x1.80mm_HandSolder" H 5588 3600 50  0001 C CNN
 F 3 "~" H 5550 3750 50  0001 C CNN
 	1    5550 3750
@@
 F 0 "C1" H 3335 3204 50  0000 R CNN
 F 1 "10uF" H 3335 3295 50  0000 R CNN
-F 2 "Capacitor_SMD:C_0805_2012Metric_Pad1.15x1.40mm_HandSolder" H 3488 3100 50  0001 C CNN
+F 2 "Capacitor_SMD:C_1206_3216Metric_Pad1.33x1.80mm_HandSolder" H 3488 3100 50  0001 C CNN
 F 3 "~" H 3450 3250 50  0001 C CNN
 	1    3450 3250
@@
 F 0 "FB1" V 2863 3100 50  0000 C CNN
 F 1 "Ferrite_Bead_Small" V 2954 3100 50  0000 C CNN
-F 2 "Resistor_SMD:R_0805_2012Metric_Pad1.15x1.40mm_HandSolder" V 3030 3100 50  0001 C CNN
+F 2 "Resistor_SMD:R_1206_3216Metric_Pad1.30x1.75mm_HandSolder" V 3030 3100 50  0001 C CNN
 F 3 "~" H 3100 3100 50  0001 C CNN
 	1    3100 3100
