File: TBM930_De-ice_panel/TBM930_De-ice_panel.kicad_pcb (KiCad board)
At the start: 2 copper layers, 190.5 x 101.6 mm, 91 parts, among them J1 SW_AIRFRAME_DE_ICE, J10 AVR-ISP-6, J11 Screw_Terminal_01x02, J2 SW_ICE_LIGHT, J3 SW_PROP_DE_ICE, J4 SW_WIND_SHIELD, J5 SW_PITOT_L_HTR, J6 SW_PITOT_R_HTR, J7 SW_INERT_SEP, J8 Barrel_Jack, J9 USB_B_Mini, SW1 SW_Push, SW2 SW_Push, U1 TLC5917IN, U2 TLC5917IN, U3 ATmega32U4-MU, Y1 Crystal_GND24

Commit message: Fix PCB holes
Parts:
- HOLE1, HOLE2, HOLE3, HOLE4: value MountingHole_3.2mm_M3 -> MountingHole
- TH1, TH2, TH3: value JLCPCB_Tooling_Hole -> MountingHole
- TSW1, TSW2, TSW3, TSW4, TSW5, TSW6, TSW7: value Mini toggle - SPDT -> MountingHole
