File: TBM930_De-ice_panel/TBM930_De-ice_panel.sch (KiCad schematic (older format))
At the start: 91 parts, among them J1 SW_AIRFRAME_DE_ICE, J10 AVR-ISP-6, J11 Screw_Terminal_01x02, J2 SW_ICE_LIGHT, J3 SW_PROP_DE_ICE, J4 SW_WIND_SHIELD, J5 SW_PITOT_L_HTR, J6 SW_PITOT_R_HTR, J7 SW_INERT_SEP, J8 Barrel_Jack, J9 USB_B_Mini, SW1 SW_Push, SW2 SW_Push, U1 TLC5917IN, U2 TLC5917IN, U3 ATmega32U4-MU, Y1 Crystal_GND24

Commit message: Change footprint for terminal block
Parts:
- J11: footprint TerminalBlock_Philmore:TerminalBlock_Philmore_TB132_1x02_P5.00mm_Horizontal -> TerminalBlock_Phoenix:TerminalBlock_Phoenix_PT-1,5-2-5.0-H_1x02_P5.00mm_Horizontal
Changed lines of the file:
@@
 F 0 "J11" H 4400 5250 50  0000 R CNN
 F 1 "Screw_Terminal_01x02" H 4600 5350 50  0000 R CNN
-F 2 "TerminalBlock_Philmore:TerminalBlock_Philmore_TB132_1x02_P5.00mm_Horizontal" H 4350 5550 50  0001 C CNN
+F 2 "TerminalBlock_Phoenix:TerminalBlock_Phoenix_PT-1,5-2-5.0-H_1x02_P5.00mm_Horizontal" H 4350 5550 50  0001 C CNN
 F 3 "~" H 4350 5550 50  0001 C CNN
 	1    4350 5550
